File: DMH_VCA_Bank_PCB_1/Power.kicad_sch (KiCad schematic)
At the start: 14 parts, among them J100 IDC_02x05, U1 TL074, U2 TL074, U3 TL074

Commit message: KiCad 10 and updated SynthStuff
Parts:
- D1: value SB140+ -> SB140; symbol SynthStuff:Power_Bus_Schotty_+ -> Diode:SB140
- D2: value SB140- -> SB140; symbol SynthStuff:Power_Bus_Schotty_- -> Diode:SB140
