File: DMH_VCA_Bank_PCB_1/VCA_B.kicad_sch (KiCad schematic)
At the start: 22 parts, among them Q3 BC548, Q4 BC548, U1 TL074, U2 TL074

Commit message: Finished schematic of PCB 1
Parts:
- renumbered U2 to U1, U1 to U2
Connections:
- net CV Amt B Pot: now also U2.3 (+); no longer U2.12 (+)
- net GND: now also U2.5 (+); no longer U2.10 (+)
- net at R18.1, R20.2: now also U1.14; no longer U1.1
- net at R18.2, R19.1: now also U1.13 (-); no longer U1.2 (-)
- net at R64.1, RV11.2, RV11.3: now also U2.1; no longer U2.14
- net at R29.1, R30.2, R64.2: now also U2.6 (-); no longer U2.9 (-)
- net at R21.1, R22.1: now also U1.12 (+); no longer U1.3 (+)
- net at R13.2, RV11.1: now also U2.2 (-); no longer U2.13 (-)
- net at R27.1, R29.2: now also U2.7; no longer U2.8
Changed lines of the file:
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@@
 		(at 234.95 76.2 0)
 		(mirror x)
-		(unit 1)
-		(exclude_from_sim no)
-		(in_bom yes)
-		(on_board yes)
-		(dnp no)
-		(property "Reference" "U2"
+		(unit 4)
+		(exclude_from_sim no)
+		(in_bom yes)
+		(on_board yes)
+		(dnp no)
+		(property "Reference" "U1"
 			(at 234.95 86.36 0)
 			(effects
@@
 			(project "DMH_Tripple_VCA_PCB_1"
 				(path "/58f4306d-5387-4983-bb08-41a2313fd315/b1c4e848-8fe8-4310-abec-b04b02b54b3f"
-					(reference "U2")
-					(unit 1)
+					(reference "U1")
+					(unit 4)
 				)
 			)
@@
 		(at 138.43 152.4 0)
 		(mirror x)
-		(unit 3)
-		(exclude_from_sim no)
-		(in_bom yes)
-		(on_board yes)
-		(dnp no)
-		(property "Reference" "U1"
+		(unit 2)
+		(exclude_from_sim no)
+		(in_bom yes)
+		(on_board yes)
+		(dnp no)
+		(property "Reference" "U2"
 			(at 138.43 162.56 0)
 			(effects
@@
 			(project "DMH_Tripple_VCA_PCB_1"
 				(path "/58f4306d-5387-4983-bb08-41a2313fd315/b1c4e848-8fe8-4310-abec-b04b02b54b3f"
-					(reference "U1")
-					(unit 3)
+					(reference "U2")
+					(unit 2)
 				)
 			)
@@
 		(at 88.9 139.7 0)
 		(mirror x)
-		(unit 4)
+		(unit 1)
 		(exclude_from_sim no)
 		(in_bom yes)
@@
 				(path "/58f4306d-5387-4983-bb08-41a2313fd315/b1c4e848-8fe8-4310-abec-b04b02b54b3f"
 					(reference "U2")
-					(unit 4)
-				)
-			)
+					(unit 1)
+				)
+			)
