File: DMH_VCA_Bank_PCB_1/DMH_VCA_Bank_PCB_1.kicad_pcb (KiCad board)
At the start: 2 copper layers, 48 x 175 mm, 95 parts, among them J1 TS_Jack_6.35mm_Sw, J10 TS_Jack_6.35mm_Sw, J100 IDC_02x05, J2 TS_Jack_6.35mm_Sw, J200 IDC_02x05, J3 TS_Jack_6.35mm_Sw, J4 TS_Jack_6.35mm_Sw, J5 TS_Jack_6.35mm_Sw, J50 Conn_01x08, J6 TS_Jack_6.35mm_Sw, J60 Conn_01x08, J7 TS_Jack_6.35mm_Sw, J70 Conn_01x08, J8 TS_Jack_6.35mm_Sw, J9 TS_Jack_6.35mm_Sw, Q1 BC548, Q2 BC548, Q3 BC548, Q4 BC548, Q5 BC548, Q6 BC548, U1 TL074, U2 TL074, U3 TL074

Commit message: PCB 1 placement started
Parts:
- removed C1, C2: 47uF, Capacitor_THT:CP_Radial_D5.0mm_P2.00mm
- removed C3, C4, C5, C6, C7, C8: 100nF, Capacitor_THT:C_Disc_D4.3mm_W1.9mm_P5.00mm
- removed D1: SB140+, Diode_THT:D_DO-41_SOD81_P10.16mm_Horizontal
- removed D2: SB140-, Diode_THT:D_DO-41_SOD81_P10.16mm_Horizontal
- removed J1, J10, J2, J3, J4, J5, J6, J7, J8, J9: TS_Jack_6.35mm_Sw, SynthStuff:CUI_MJ-63052A
- removed J100: IDC_02x05, SynthStuff:IDC-Header_2x05_P2.54mm_Vertical_Eurorack
- removed J200: IDC_02x05, SynthStuff:IDC-Header_2x05_P2.54mm_Vertical_BackBone
- removed J50, J60, J70: Conn_01x08, Connector_PinSocket_2.54mm:PinSocket_1x08_P2.54mm_Vertical
- removed Q1, Q2, Q3, Q4, Q5, Q6: BC548, Package_TO_SOT_THT:TO-92L_Inline_Wide
- removed R1, R16, R17, R2, R31, R32: 20k, Resistor_THT:R_Axial_DIN0207_L6.3mm_D2.5mm_P2.54mm_Vertical
- removed R10, R11, R25, R26, R40, R41: 100R, Resistor_THT:R_Axial_DIN0207_L6.3mm_D2.5mm_P2.54mm_Vertical
- removed R12, R19, R21, R27, R34, R36, R4, R42, R6: 10k, Resistor_THT:R_Axial_DIN0207_L6.3mm_D2.5mm_P2.54mm_Vertical
- removed R13, R28, R62: 33k, Resistor_THT:R_Axial_DIN0207_L6.3mm_D2.5mm_P2.54mm_Vertical
- removed R14, R15, R18, R22, R23, R24, R29, R3, R30, R33, R37, R38, R39, R44, R45, R46, R47, R48, R49, R50, R51, R63, R64, R65, R7, R8, R9: 100k, Resistor_THT:R_Axial_DIN0207_L6.3mm_D2.5mm_P2.54mm_Vertical
- removed R20, R35, R5, R52: 1k, Resistor_THT:R_Axial_DIN0207_L6.3mm_D2.5mm_P2.54mm_Vertical
- removed RV1, RV2, RV3: 100k, Potentiometer_THT:Potentiometer_Bourns_3296W_Vertical
- removed RV10, RV11, RV12: 50k, Potentiometer_THT:Potentiometer_Bourns_3296W_Vertical
- removed U1, U2, U3: TL074, Package_DIP:DIP-14_W7.62mm_Socket
Routing:
- net +12V: track 242.4 -> 0.00 mm
- net /Inputs and Outputs/Mute A Switch: track 165.6 -> 0.00 mm
- net /Inputs and Outputs/CV B Jack: track 155.7 -> 0.00 mm
- net /Inputs and Outputs/Output B Jack: track 154.0 -> 0.00 mm
- net -12V: track 152.4 -> 0.00 mm
- net /Inputs and Outputs/Output A Jack: track 143.8 -> 0.00 mm
- net /Inputs and Outputs/CV A Jack: track 120.0 -> 0.00 mm
- net /Inputs and Outputs/Input B Jack: track 119.8 -> 0.00 mm
- net /Inputs and Outputs/Output C Jack: track 118.4 -> 0.00 mm
- net /Inputs and Outputs/Input A Jack: track 113.9 -> 0.00 mm
- net /Inputs and Outputs/CV C Jack: track 112.0 -> 0.00 mm
- net /Inputs and Outputs/Input C Jack: track 101.5 -> 0.00 mm
- net Net-(U2A--): track 97.8 -> 0.00 mm
- net Net-(J200-Pin_9): track 87.1 -> 0.00 mm
- net Net-(R39-Pad1): track 64.2 -> 0.00 mm
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