File: DMH_VCA_Bank_PCB_1/DMH_VCA_Bank_PCB_1.kicad_pcb (KiCad board)
At the start: 2 copper layers, 48 x 175 mm, 111 parts, among them J1 TS_Jack_6.35mm_Sw, J10 TS_Jack_6.35mm_Sw, J100 IDC_02x05, J11 TS_Jack_6.35mm_Sw, J12 TS_Jack_6.35mm_Sw, J2 TS_Jack_6.35mm_Sw, J200 IDC_02x08, J3 TS_Jack_6.35mm_Sw, J4 TS_Jack_6.35mm_Sw, J5 TS_Jack_6.35mm_Sw, J50 Conn_01x06, J6 TS_Jack_6.35mm_Sw, J60 Conn_01x06, J7 TS_Jack_6.35mm_Sw, J70 Conn_01x06, J8 TS_Jack_6.35mm_Sw, J80 Conn_01x06, J9 TS_Jack_6.35mm_Sw, Q1 BC548, Q2 BC548, Q3 BC548, Q4 BC548, Q5 BC548, Q6 BC548, Q7 BC548, Q8 BC548, U1 TL074, U2 TL074, U3 TL074

Commit message: KiCad 10 and updated SynthStuff
Parts:
- D1: value SB140+ -> SB140
- D2: value SB140- -> SB140
Routing:
- net /Inputs and Outputs/CV A Jack: track 126.6 -> 127.3 mm
