File: DMH_VCA_Bank_PCB_2/Inputs_and_Outputs.kicad_sch (KiCad schematic)
At the start: 36 parts, among them J0 Conn_01x01, J1 TS_Jack_6.35mm_Sw, J10 TS_Jack_6.35mm_Sw, J2 TS_Jack_6.35mm_Sw, J200 IDC_02x05, J3 TS_Jack_6.35mm_Sw, J4 TS_Jack_6.35mm_Sw, J5 TS_Jack_6.35mm_Sw, J50 Conn_01x08, J6 TS_Jack_6.35mm_Sw, J60 Conn_01x08, J7 TS_Jack_6.35mm_Sw, J70 Conn_01x08, J8 TS_Jack_6.35mm_Sw, J9 TS_Jack_6.35mm_Sw, SW1 SW_DPDT, SW2 SW_DPDT, SW3 SW_DPDT

Commit message: Finished schematic of PCB 1
Parts:
- removed D3, D4, D5: LED_Dual_AKA, SynthStuff:LED_D3.0mm-2color, symbol Device:LED_Dual_AKA
- removed R56, R57, R58, R59, R60, R61: 1k, Resistor_THT:R_Axial_DIN0207_L6.3mm_D2.5mm_P7.62mm_Horizontal, symbol Device:R_US
- removed SW1, SW2, SW3: SW_DPDT, SynthStuff:Toggle_Switch_2_Poles_TE, symbol SynthStuff:Switch_DPDT
- J2: Function Output A -> CV A
- J3: Function CV A -> Output A
- J5: Function Output B -> CV B
- J6: Function CV B -> Output B
- J8: Function Output C -> CV C
- J9: Function CV C -> Output C
Connections:
- net GND: no longer J0.1 (Pin_1)
- no-connect marks 4 -> 1
