File: DMH_VCA_Bank_PCB_2/DMH_VCA_Bank_PCB_2.kicad_pcb (KiCad board)
At the start: 2 copper layers, 48 x 124.5 mm, 25 parts, among them J0 Conn_01x01, J50 Conn_01x08, J60 Conn_01x08, J70 Conn_01x08, SW1 SW_DPDT, SW2 SW_DPDT, SW3 SW_DPDT

Commit message: Finished PCB 2
Parts:
- removed D3, D4, D5: LED_Dual_AKA, SynthStuff:LED_D3.0mm-2color
- removed R57, R58, R59, R60, R61: 1k, Resistor_THT:R_Axial_DIN0207_L6.3mm_D2.5mm_P7.62mm_Horizontal
- removed SW1, SW2, SW3: SW_DPDT, SynthStuff:Toggle_Switch_2_Poles_TE
- added J80: Conn_01x06, Connector_PinSocket_2.54mm:PinSocket_1x06_P2.54mm_Vertical, B.Cu at (97.0, 132.0)
- added RV13: 100k, SynthStuff:Potentiometer_TT_P110KH1, F.Cu at (85.0, 148.0)
- added RV14: 100k, SynthStuff:Potentiometer_Alpha_RD901F-40-00D_Single_Vertical, F.Cu at (60.0, 144.5)
- J50, J60, J70: value Conn_01x08 -> Conn_01x06; footprint Connector_PinHeader_2.54mm:PinHeader_1x08_P2.54mm_Vertical -> Connector_PinSocket_2.54mm:PinSocket_1x06_P2.54mm_Vertical
- R56: value 1k -> 20k
- moved R56 64.5 mm to (58.7, 128.5), turned to 0 degrees
- moved J70 53.3 mm to (53.0, 103.0)
- moved J60 46.6 mm to (97.0, 77.0)
- moved R55 46.4 mm to (58.7, 101.0), turned to 0 degrees
- moved J50 46.3 mm to (53.0, 48.0)
- moved R54 45.3 mm to (58.7, 73.5), turned to 0 degrees
- moved R53 44.2 mm to (58.7, 46.0), turned to 0 degrees
- moved RV9 39.8 mm to (85.0, 120.5)
- moved RV8 38.5 mm to (85.0, 93.0)
- moved RV7 37.2 mm to (85.0, 65.5)
- moved RV6 25.2 mm to (60.0, 117.0)
- moved RV5 24.0 mm to (60.0, 89.5)
- moved RV4 22.8 mm to (60.0, 62.0)
- moved J0 20.0 mm to (97.0, 120.0)
Connections:
- J50 pad 2: /Inputs and Outputs/Mute A Switch -> /Inputs and Outputs/Offset A Pot
- J50 pad 3: /Inputs and Outputs/Output A Jack -> /Inputs and Outputs/CV Amt A Pot
- J50 pad 4: /Inputs and Outputs/Offset A Pot -> /Inputs and Outputs/CV A Jack
- J50 pad 5: /Inputs and Outputs/CV Amt A Pot -> GND
- J50 pad 6: /Inputs and Outputs/CV A Jack -> GND
- J60 pad 2: /Inputs and Outputs/Mute B Switch -> /Inputs and Outputs/Offset B Pot
- J60 pad 3: /Inputs and Outputs/Output B Jack -> /Inputs and Outputs/CV Amt B Pot
- J60 pad 4: /Inputs and Outputs/Offset B Pot -> /Inputs and Outputs/CV B Jack
- J60 pad 5: /Inputs and Outputs/CV Amt B Pot -> GND
- J60 pad 6: /Inputs and Outputs/CV B Jack -> GND
- J70 pad 2: /Inputs and Outputs/Mute C Switch -> /Inputs and Outputs/Offset C Pot
- J70 pad 3: /Inputs and Outputs/Output C Jack -> /Inputs and Outputs/CV Amt C Pot
- J70 pad 4: /Inputs and Outputs/Offset C Pot -> /Inputs and Outputs/CV C Jack
- J70 pad 5: /Inputs and Outputs/CV Amt C Pot -> GND
- J70 pad 6: /Inputs and Outputs/CV C Jack -> GND
- R56 pad 2: Net-(R56-Pad2) -> +12V
Routing:
- net /Inputs and Outputs/Mute C Switch: track 98.6 -> 0.00 mm
- net /Inputs and Outputs/Output C Jack: track 93.6 -> 0.00 mm
- net /Inputs and Outputs/Output B Jack: track 88.0 -> 0.00 mm
- net /Inputs and Outputs/Mute B Switch: track 77.0 -> 0.00 mm
- net /Inputs and Outputs/Offset A Pot: track 84.4 -> 17.4 mm
- net Net-(R57-Pad2): track 47.2 -> 0.00 mm
- net /Inputs and Outputs/Output A Jack: track 46.1 -> 0.00 mm
- net /Inputs and Outputs/Mute A Switch: track 45.9 -> 0.00 mm
- net /Inputs and Outputs/Offset D Pot: track 0.00 -> 38.6 mm
- net Net-(R59-Pad2): track 36.3 -> 0.00 mm
- net Net-(R61-Pad2): track 35.5 -> 0.00 mm
- net /Inputs and Outputs/CV B Jack: track 43.7 -> 11.8 mm
- net +12V: track 217.6 -> 185.7 mm
- net /Inputs and Outputs/CV Amt B Pot: track 45.6 -> 15.4 mm
- net /Inputs and Outputs/CV C Jack: track 21.3 -> 46.4 mm
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Other:
- board size 48 x 124.5 mm -> 48 x 108 mm
- board text added: "Mk1.0 - Month 2025"
- board text removed: "Mk2.0 - Month 2025"
