File: DMH_VCA_Bank_PANEL/DMH_VCA_Bank_PANEL.kicad_pcb (KiCad board)
At the start: 2 copper layers, 50 x 200 mm, 19 parts, among them J0 Panel_GND_Solder_Wire_Pad

Commit message: Panel ready
Parts:
- added H19: Offset D, SynthStuff:Pot_Cutout_Tiny, F.Cu at (62.5, 137.0)
- added H20: CV D Amt, SynthStuff:Pot_Cutout_Tiny_attv_P110KH1, F.Cu at (87.5, 137.0)
- added H21: In D, SynthStuff:Jack_6.35mm_Cutout_v3, F.Cu at (58.5, 208.8)
- added H22: CV D, SynthStuff:Jack_6.35mm_Cutout_v3, F.Cu at (75.0, 208.8)
- added H23: Out C, SynthStuff:Jack_6.35mm_Cutout_Output_v6, F.Cu at (91.5, 192.2)
- added H24: Out D, SynthStuff:Jack_6.35mm_Cutout_Output_v6, F.Cu at (91.5, 208.8)
- H10: value CV 2 -> CV C Amt; footprint SynthStuff:Jack_6.35mm_Cutout_v3 -> SynthStuff:Pot_Cutout_Tiny_attv_P110KH1
- H11: value Output -> Out A
- H12: value Offset -> Offset B; footprint SynthStuff:Pot_Cutout_Small -> SynthStuff:Pot_Cutout_Tiny
- H13: value CV 1 Amt -> CV B Amt
- H14: value CV 2 Amt -> In C; footprint SynthStuff:Pot_Cutout_Tiny_attv_P110KH1 -> SynthStuff:Jack_6.35mm_Cutout_v3
- H15: value Input -> In B
- H16: value Output -> Out B
- H17: value CV 1 -> CV B
- H18: value CV 2 -> CV C
- H5: value Offset -> Offset A; footprint SynthStuff:Pot_Cutout_Small -> SynthStuff:Pot_Cutout_Tiny
- H6: value CV 1 Amt -> CV A Amt
- H7: value CV 2 Amt -> Offset C; footprint SynthStuff:Pot_Cutout_Tiny_attv_P110KH1 -> SynthStuff:Pot_Cutout_Tiny
- H8: value Input -> In A
- H9: value CV 1 -> CV A
- moved H8 108.5 mm to (58.5, 159.2)
- moved H13 104.0 mm to (87.5, 82.0)
- moved H11 95.9 mm to (91.5, 159.2)
- moved H12 71.7 mm to (62.5, 82.0)
- moved H6 47.5 mm to (87.5, 54.5)
- moved H9 43.0 mm to (75.0, 159.2)
- moved H16 36.6 mm to (91.5, 175.8)
- moved H17 35.1 mm to (75.0, 175.8)
- moved H15 34.2 mm to (58.5, 175.8)
- moved H7 28.3 mm to (62.5, 109.5)
- moved H5 21.2 mm to (62.5, 54.5)
- moved H18 20.4 mm to (75.0, 192.2)
- moved H10 8.51 mm to (87.5, 109.5)
- moved H14 7.70 mm to (58.5, 192.2)
- moved J0 5.00 mm to (95.0, 125.0)
Other:
- board text added: "074-4"
- board text removed: "074-2"

Commit message: Generated Gerbers
Other:
- board text added: "Mk1.0 - October 2025"
- board text removed: "Mk1.0 - March 2025"
Changed lines of the file:
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@@
 			(psa4output no)
 			(plot_black_and_white yes)
-			(plotinvisibletext no)
 			(sketchpadsonfab no)
 			(plotpadnumbers no)
@@
 			)
 		)
-		(property "Datasheet" ""
+		(property "Datasheet" "~"
 			(at 0 0 0)
 			(unlocked yes)
@@
 			)
 		)
-		(property "Datasheet" ""
+		(property "Datasheet" "~"
 			(at 0 0 0)
 			(unlocked yes)
@@
 			)
 		)
-		(property "Datasheet" ""
+		(property "Datasheet" "~"
 			(at 0 0 0)
 			(unlocked yes)
@@
 			)
 		)
-		(property "Datasheet" ""
+		(property "Datasheet" "~"
 			(at 0 0 0)
 			(unlocked yes)
@@
 			)
 		)
-		(property "Datasheet" ""
+		(property "Datasheet" "~"
 			(at 0 0 0)
 			(unlocked yes)
@@
 			)
 		)
-		(property "Datasheet" ""
+		(property "Datasheet" "~"
 			(at 0 0 0)
 			(unlocked yes)
@@
 			)
 		)
-		(property "Datasheet" ""
+		(property "Datasheet" "~"
 			(at 0 0 0)
 			(unlocked yes)
@@
 			)
 		)
-		(property "Datasheet" ""
+		(property "Datasheet" "~"
 			(at 0 0 0)
 			(unlocked yes)
@@
 			)
 		)
-		(property "Datasheet" ""
+		(property "Datasheet" "~"
 			(at 0 0 0)
 			(unlocked yes)
@@
 			)
 		)
-		(property "Datasheet" ""
+		(property "Datasheet" "~"
 			(at 0 0 0)
 			(unlocked yes)
@@
 			)
 		)
-		(property "Datasheet" ""
+		(property "Datasheet" "~"
 			(at 0 0 0)
 			(unlocked yes)
@@
 			)
 		)
-		(property "Datasheet" ""
+		(property "Datasheet" "~"
 			(at 0 0 0)
 			(unlocked yes)
@@
 			)
 		)
-		(property "Datasheet" ""
+		(property "Datasheet" "~"
 			(at 0 0 0)
 			(unlocked yes)
@@
 			)
 		)
-		(property "Datasheet" ""
+		(property "Datasheet" "~"
 			(at 0 0 0)
 			(unlocked yes)
@@
 			)
 		)
-		(property "Datasheet" ""
+		(property "Datasheet" "~"
 			(at 0 0 0)
 			(unlocked yes)
@@
 			)
 		)
-		(property "Datasheet" ""
+		(property "Datasheet" "~"
 			(at 0 0 0)
 			(unlocked yes)
@@
 			)
 		)
-		(property "Datasheet" ""
+		(property "Datasheet" "~"
 			(at 0 0 0)
 			(unlocked yes)
@@
 			)
 		)
-		(property "Datasheet" ""
+		(property "Datasheet" "~"
 			(at 0 0 0)
 			(unlocked yes)
@@
 			)
 		)
-		(property "Datasheet" ""
+		(property "Datasheet" "~"
 			(at 0 0 0)
 			(unlocked yes)
@@
 			)
 		)
-		(property "Datasheet" ""
+		(property "Datasheet" "~"
 			(at 0 0 0)
 			(unlocked yes)
@@
 			)
 		)
-		(property "Datasheet" ""
+		(property "Datasheet" "~"
 			(at 0 0 0)
 			(unlocked yes)
@@
 			)
 		)
-		(property "Datasheet" ""
+		(property "Datasheet" "~"
 			(at 0 0 0)
 			(unlocked yes)
@@
 			)
 		)
-		(property "Datasheet" ""
+		(property "Datasheet" "~"
 			(at 0 0 0)
 			(unlocked yes)
@@
 			)
 		)
-		(property "Datasheet" ""
+		(property "Datasheet" "~"
 			(at 0 0 0)
 			(unlocked yes)
@@
 			)
 		)
-		(property "Datasheet" ""
+		(property "Datasheet" "~"
 			(at 0 0 0)
 			(unlocked yes)
@@
 			(polygon
 				(pts
-					(xy 63.647593 38.801891) (xy 63.868032 39.20824) (xy 64.131234 39.543203) (xy 64.439033 39.80781)
-					(xy 64.793263 40.003088) (xy 65.195757 40.130067) (xy 65.648349 40.189774) (xy 65.843824 40.195052)
-					(xy 66.31946 40.161965) (xy 66.740892 40.062018) (xy 67.111162 39.894183) (xy 67.433311 39.657431)
-					(xy 67.71038 39.350734) (xy 67.94541 38.973062) (xy 68.028332 38.801891) (xy 70.738451 32.779839)
-					(xy 70.861549 32.441807) (xy 68.497279 32.441807) (xy 68.407397 32.711451) (xy 66.168179 37.959741)
-					(xy 65.853594 38.196168) (xy 65.52924 37.959741) (xy 63.266574 32.711451) (xy 63.188416 32.441807)
-					(xy 60.790928 32.441807) (xy 60.914027 32.779839)
+					(xy 63.64857 38.839016) (xy 63.794353 39.122984) (xy 63.959816 39.373672) (xy 64.132303 39.577694)
+					(xy 64.322862 39.753342) (xy 64.524506 39.896302) (xy 64.743865 40.013279) (xy 65.240116 40.170779)
+					(xy 65.843824 40.226315) (xy 66.178355 40.210627) (xy 66.486496 40.163337) (xy 66.748894 40.091171)
+					(xy 66.990389 39.991411) (xy 67.203469 39.869327) (xy 67.39871 39.721286) (xy 67.739744 39.344695)
+					(xy 68.027355 38.839016) (xy 70.737963 32.840411) (xy 70.861061 32.504333) (xy 68.497767 32.504333)
+					(xy 68.408374 32.773) (xy 66.168179 37.999309) (xy 66.098945 38.119832) (xy 66.018246 38.193425)
+					(xy 65.854571 38.23427) (xy 65.745722 38.217896) (xy 65.647979 38.165801) (xy 65.530217 37.999309)
+					(xy 63.267551 32.773) (xy 63.189393 32.504333) (xy 60.792394 32.504333) (xy 60.915492 32.840411)
 				)
 			)
 			(polygon
 				(pts
-					(xy 78.515143 38.076978) (xy 74.550593 38.076978) (xy 74.11308 38.045361) (xy 73.689571 37.936626)
-					(xy 73.340297 37.758351) (xy 73.026518 37.484933) (xy 72.788746 37.15553) (xy 72.629184 36.774034)
-					(xy 72.55964 36.354757) (xy 72.557572 36.267627) (xy 72.606331 35.846507) (xy 72.745478 35.456947)
-					(xy 72.96432 35.113813) (xy 73.116399 34.948715) (xy 73.455885 34.696766) (xy 73.834909 34.538911)
-					(xy 74.24844 34.462369) (xy 74.550593 34.448506) (xy 78.515143 34.448506) (xy 78.515143 32.441807)
-					(xy 74.550593 32.441807) (xy 74.107228 32.459385) (xy 73.692416 32.510989) (xy 73.305218 32.594924)
-					(xy 72.858624 32.742729) (xy 72.451878 32.935094) (xy 72.083146 33.168712) (xy 71.750593 33.440272)
-					(xy 71.420079 33.787663) (xy 71.134877 34.176351) (xy 70.899371 34.601551) (xy 70.749691 34.964782)
-					(xy 70.636866 35.345869) (xy 70.563138 35.74236) (xy 70.530753 36.151805) (xy 70.529379 36.255903)
-					(xy 70.55592 36.722989) (xy 70.633516 37.171354) (xy 70.759126 37.597733) (xy 70.929708 37.998862)
-					(xy 71.142222 38.371476) (xy 71.393627 38.712311) (xy 71.504397 38.839016) (xy 71.851943 39.174083)
-					(xy 72.245151 39.462193) (xy 72.593465 39.656165) (xy 72.972497 39.815448) (xy 73.38291 39.93798)
-					(xy 73.825368 40.0217) (xy 74.300536 40.064547) (xy 74.550593 40.07) (xy 78.515143 40.07)
+					(xy 78.515632 38.076489) (xy 74.551082 38.076489) (xy 74.238813 38.061173) (xy 73.957777 38.016485)
+					(xy 73.713366 37.946842) (xy 73.495257 37.853056) (xy 73.131745 37.599887) (xy 73.027983 37.495191)
+					(xy 72.880884 37.314063) (xy 72.758326 37.11362) (xy 72.66309 36.897664) (xy 72.596965 36.668114)
+					(xy 72.557572 36.298401) (xy 72.617675 35.839522) (xy 72.795679 35.407933) (xy 72.926223 35.212281)
+					(xy 73.080994 35.036515) (xy 73.117376 35.001472) (xy 73.310208 34.845054) (xy 73.530034 34.714905)
+					(xy 73.749126 34.625009) (xy 73.99757 34.559525) (xy 74.551082 34.509567) (xy 78.515632 34.509567)
+					(xy 78.515632 32.504333) (xy 74.551082 32.504333) (xy 74.135563 32.519731) (xy 73.745022 32.564991)
+					(xy 73.382202 32.637849) (xy 73.042396 32.737247) (xy 72.723728 32.862337) (xy 72.426768 33.01142)
+					(xy 71.884644 33.384657) (xy 71.751082 33.501332) (xy 71.28893 34.014118) (xy 71.094042 34.300285)
+					(xy 70.925293 34.604164) (xy 70.78575 34.920325) (xy 70.674919 35.250473) (xy 70.595627 35.586247)
+					(xy 70.546945 35.932325) (xy 70.530356 36.287655) (xy 70.591078 36.977622) (xy 70.770515 37.63504)
+					(xy 71.063227 38.244697) (xy 71.460538 38.788711) (xy 71.504885 38.838039) (xy 71.747993 39.081385)
+					(xy 72.014068 39.301548) (xy 72.292157 39.490111) (xy 72.592333 39.654543) (xy 72.90745 39.790681)
+					(xy 73.244434 39.901294) (xy 73.600788 39.984615) (xy 73.979415 40.040409) (xy 74.551082 40.07)
+					(xy 78.515632 40.07)
 				)
 			)
 			(polygon
 				(pts
-					(xy 84.341772 32.32214) (xy 84.790294 32.382856) (xy 85.19006 32.511397) (xy 85.542635 32.708167)
-					(xy 85.849585 32.973567) (xy 86.112474 33.308) (xy 86.332868 33.71187) (xy 89.066434 39.726106)
-					(xy 89.189533 40.07) (xy 86.90342 40.07) (xy 86.815492 39.806217) (xy 86.411026 38.864417) (xy 81.930635 38.864417)
-					(xy 81.539847 39.794494) (xy 81.459735 40.07) (xy 79.118912 40.07) (xy 79.24201 39.726106) (xy 80.383936 37.193796)
-					(xy 82.67118 37.193796) (xy 85.672436 37.193796) (xy 84.507886 34.493447) (xy 84.49432 34.463444)
-					(xy 84.160084 34.258974) (xy 84.14748 34.259142) (xy 83.824006 34.493447) (xy 82.67118 37.193796)
-					(xy 80.383936 37.193796) (xy 81.954083 33.71187) (xy 82.036986 33.541964) (xy 82.271918 33.165917)
-					(xy 82.549104 32.859145) (xy 82.871942 32.621246) (xy 83.243832 32.451816) (xy 83.668171 32.350453)
-					(xy 84.14836 32.316755)
+					(xy 84.74036 32.372322) (xy 85.233641 32.531552) (xy 85.453141 32.650281) (xy 85.655152 32.795272)
+					(xy 85.846684 32.973631) (xy 86.020183 33.180534) (xy 86.186653 33.43427) (xy 86.333357 33.721151)
+					(xy 89.065946 39.73441) (xy 89.189044 40.07) (xy 86.904397 40.07) (xy 86.81552 39.814911) (xy 86.814515 39.812568)
+					(xy 86.411515 38.894214) (xy 81.931612 38.894214) (xy 81.539847 39.801332) (xy 81.539029 39.803513)
+					(xy 81.4612 40.07) (xy 79.120377 40.07) (xy 79.243475 39.73441) (xy 80.37462 37.225059) (xy 82.670691 37.225059)
+					(xy 85.672436 37.225059) (xy 84.507397 34.507124) (xy 84.383319 34.339506) (xy 84.278173 34.287542)
+					(xy 84.160572 34.271186) (xy 84.142955 34.271514) (xy 83.964403 34.326253) (xy 83.888062 34.398134)
+					(xy 83.824494 34.507124) (xy 82.670691 37.225059) (xy 80.37462 37.225059) (xy 81.954083 33.721151)
+					(xy 82.252465 33.197366) (xy 82.595413 32.821092) (xy 82.791321 32.673241) (xy 83.005212 32.551142)
+					(xy 83.246803 32.451603) (xy 83.509383 32.379497) (xy 83.816208 32.332413) (xy 84.149337 32.316755)
 				)
 			)
@@
 		)
 	)
-	(gr_text "Mk1.0 - March 2025"
+	(gr_text "Mk1.0 - October 2025"
 		(at 75 222.95 0)
 		(layer "B.SilkS")
