File: DMH_VCA_Bank_PANEL/DMH_VCA_Bank_PANEL.kicad_sch (KiCad schematic)
At the start: 19 parts, among them J0 Panel_GND_Solder_Wire_Pad

Commit message: Panel ready
Parts:
- removed H10: CV 2, SynthStuff:Jack_6.35mm_Cutout_v3, symbol SynthStuff:MountingHole_Jack6.35mm_v2
- removed H14: CV 2 Amt, SynthStuff:Pot_Cutout_Tiny_attv_P110KH1, symbol SynthStuff:MountingHole_Pot
- added H10: CV C Amt, SynthStuff:Pot_Cutout_Tiny_attv_P110KH1, symbol SynthStuff:MountingHole_Pot
- added H14: In C, SynthStuff:Jack_6.35mm_Cutout_v3, symbol SynthStuff:MountingHole_Jack6.35mm_v2
- added H19: Offset D, SynthStuff:Pot_Cutout_Tiny, symbol SynthStuff:MountingHole_Pot
- added H20: CV D Amt, SynthStuff:Pot_Cutout_Tiny_attv_P110KH1, symbol SynthStuff:MountingHole_Pot
- added H21: In D, SynthStuff:Jack_6.35mm_Cutout_v3, symbol SynthStuff:MountingHole_Jack6.35mm_v2
- added H22: CV D, SynthStuff:Jack_6.35mm_Cutout_v3, symbol SynthStuff:MountingHole_Jack6.35mm_v2
- added H23: Out C, SynthStuff:Jack_6.35mm_Cutout_Output_v6, symbol SynthStuff:MountingHole_Jack6.35mm_v2
- added H24: Out D, SynthStuff:Jack_6.35mm_Cutout_Output_v6, symbol SynthStuff:MountingHole_Jack6.35mm_v2
- H11: value Output -> Out A
- H12: value Offset -> Offset B; footprint SynthStuff:Pot_Cutout_Small -> SynthStuff:Pot_Cutout_Tiny
- H13: value CV 1 Amt -> CV B Amt
- H15: value Input -> In B
- H16: value Output -> Out B
- H17: value CV 1 -> CV B
- H18: value CV 2 -> CV C
- H5: value Offset -> Offset A; footprint SynthStuff:Pot_Cutout_Small -> SynthStuff:Pot_Cutout_Tiny
- H6: value CV 1 Amt -> CV A Amt
- H7: value CV 2 Amt -> Offset C; footprint SynthStuff:Pot_Cutout_Tiny_attv_P110KH1 -> SynthStuff:Pot_Cutout_Tiny
- H8: value Input -> In A
- H9: value CV 1 -> CV A
Connections:
- net GND: now also H10.1, H14.1, H19.1, H20.1, H21.1, H22.1, H23.1, H24.1
Other:
- moved on the sheet: H11, H12, H13, H15, H16, H17, H5, H6, H8, H9
